File: iotkong/iotkong.kicad_pcb (KiCad board)
At the start: 2 copper layers, 223 x 54.4 mm, 21 parts, among them J1 Conn_01x15_Female, J10 Conn_01x15_Female, J11 Conn_01x15_Female, J2 USB_B, J3 Conn_01x15_Female, J4 Conn_01x15_Female, J5 Conn_01x15_Female, J6 Conn_01x15_Female, J7 Conn_01x15_Female, J8 Conn_01x15_Female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

Commit message: silkscreening
Parts:
- added SW4: SW_SPST, Button_Switch_THT:SW_PUSH_6mm, F.Cu at (218.4, 57.9)
- added SW5: SW_SPST, Button_Switch_THT:SW_PUSH_6mm, F.Cu at (256.5, 57.9)
- moved C1 2.59 mm to (91.4, 70.6)
- moved C2 2.54 mm to (133.1, 70.1)
- moved C4 2.54 mm to (255.0, 70.1)
- moved C5 1.52 mm to (175.3, 69.6)
Routing:
- net Net-(J7-Pad3): track 17.4 -> 23.9 mm
- net Net-(J11-Pad3): track 19.2 -> 24.1 mm
Other:
- board text added: "Board 1"
- board text added: "Board 2"
- board text added: "Board 3"
- board text added: "Board 4"
- board text added: "Board 5"
- board text added: "Kevin Glavin v0.1"
- board text added: "RST 1"
- board text added: "RST 2"
- board text added: "RST 3"
- board text added: "RST 4"
- board text added: "RST 5"

Commit message: 0.98 alignment for board
Parts:
- C1, C2, C3, C4, C5: footprint Capacitor_THT:C_Disc_D4.3mm_W1.9mm_P5.00mm -> Capacitor_THT:CP_Radial_D8.0mm_P5.00mm
- J1, J10, J11, J3, J4, J5, J6, J7, J8, J9: footprint Connector_Molex:Molex_KK-254_AE-6410-15A_1x15_P2.54mm_Vertical -> Connector_PinHeader_2.54mm:PinHeader_1x15_P2.54mm_Vertical
- moved C5 119.9 mm to (294.6, 58.9), turned to 90 degrees
- moved J10 117.1 mm to (283.5, 51.3), turned to 0 degrees
- moved SW6 111.8 mm to (291.1, 42.7), turned to 0 degrees
- moved J9 64.8 mm to (209.8, 51.3), turned to 0 degrees
- moved J2 38.6 mm to (44.7, 53.4)
- moved J8 34.2 mm to (258.1, 51.3), turned to 0 degrees
- moved J6 31.6 mm to (161.5, 51.3), turned to 0 degrees
- moved SW4 28.3 mm to (194.6, 42.7), turned to 0 degrees
- moved J7 27.5 mm to (186.9, 51.3), turned to 0 degrees
- moved J11 21.8 mm to (235.2, 51.3), turned to 0 degrees
- moved J5 20.9 mm to (138.7, 51.3), turned to 0 degrees
- moved SW5 20.5 mm to (242.8, 42.7), turned to 0 degrees
- moved C2 20.1 mm to (149.9, 58.9), turned to 90 degrees
- moved C3 19.3 mm to (198.1, 58.9), turned to 90 degrees
- moved J3 18.5 mm to (90.4, 51.3), turned to 0 degrees
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Routing:
- net Net-(J11-Pad3): track 24.1 -> 31.7 mm
- net Net-(J2-Pad1): track 28.7 -> 25.9 mm
- net Net-(J3-Pad3): track 32.2 -> 30.4 mm
- net Net-(J10-Pad3): track 31.0 -> 32.3 mm
- net Net-(J5-Pad3): track 28.9 -> 30.1 mm
- net Net-(R1-Pad1): track 9.92 -> 9.21 mm
- net Net-(J7-Pad3): track 23.9 -> 23.3 mm
- added copper zone on B.Cu, net GND
- added copper zone on F.Cu, net VCC
- removed copper zone on F.Cu, net GND
- removed copper zone on B.Cu, net VCC
Other:
- board size 223 x 54.4 mm -> 264.2 x 52.8 mm
- net class power removed
- rule pad_to_mask_clearance: 0.2 -> 0
- board text removed: "Board 1"
- board text removed: "Board 2"
- board text removed: "Board 3"
- board text removed: "Board 4"
- board text removed: "Board 5"
- board text removed: "RST 1"
- board text removed: "RST 2"
- board text removed: "RST 3"
- board text removed: "RST 4"
- board text removed: "RST 5"

Commit message: added leds and placed
Parts:
- added C10: 0.1uF, Capacitor_THT:C_Disc_D3.0mm_W1.6mm_P2.50mm, F.Cu at (284.9, 51.2)
- added C6: 0.1uF, Capacitor_THT:C_Disc_D3.0mm_W1.6mm_P2.50mm, F.Cu at (91.8, 51.1)
- added C7: 0.1uF, Capacitor_THT:C_Disc_D3.0mm_W1.6mm_P2.50mm, F.Cu at (139.9, 51.1)
- added C8: 0.1uF, Capacitor_THT:C_Disc_D3.0mm_W1.6mm_P2.50mm, F.Cu at (188.3, 51.2)
- added C9: 0.1uF, Capacitor_THT:C_Disc_D3.0mm_W1.6mm_P2.50mm, F.Cu at (236.9, 51.4)
- added D1: LED, LED_THT:LED_D5.0mm, F.Cu at (55.9, 85.3)
- added D10: LED, LED_THT:LED_D5.0mm, F.Cu at (251.0, 78.7)
- added D2: LED, LED_THT:LED_D5.0mm, F.Cu at (55.9, 78.7)
- added D3: LED, LED_THT:LED_D5.0mm, F.Cu at (105.2, 85.3)
- added D4: LED, LED_THT:LED_D5.0mm, F.Cu at (105.2, 78.7)
- added D5: LED, LED_THT:LED_D5.0mm, F.Cu at (153.4, 85.3)
- added D6: LED, LED_THT:LED_D5.0mm, F.Cu at (153.4, 78.7)
- added D7: LED, LED_THT:LED_D5.0mm, F.Cu at (201.7, 85.3)
- added D8: LED, LED_THT:LED_D5.0mm, F.Cu at (201.7, 78.7)
- added D9: LED, LED_THT:LED_D5.0mm, F.Cu at (251.0, 85.3)
- added MH1: MountingHole, MountingHole:MountingHole_3.2mm_M3_ISO7380, F.Cu at (43.2, 43.2)
- added MH2: MountingHole, MountingHole:MountingHole_3.2mm_M3_ISO7380, F.Cu at (43.2, 86.4)
- added MH3: MountingHole, MountingHole:MountingHole_3.2mm_M3_ISO7380, F.Cu at (301.0, 41.9)
- added MH4: MountingHole, MountingHole:MountingHole_3.2mm_M3_ISO7380, F.Cu at (301.0, 86.4)
- added R10: 100, Resistor_THT:R_Axial_DIN0204_L3.6mm_D1.6mm_P5.08mm_Horizontal, F.Cu at (247.9, 83.3)
- added R11: 100, Resistor_THT:R_Axial_DIN0204_L3.6mm_D1.6mm_P5.08mm_Horizontal, F.Cu at (247.9, 79.8)
- added R2: 100, Resistor_THT:R_Axial_DIN0204_L3.6mm_D1.6mm_P5.08mm_Horizontal, F.Cu at (52.3, 83.3)
- added R3: 100, Resistor_THT:R_Axial_DIN0204_L3.6mm_D1.6mm_P5.08mm_Horizontal, F.Cu at (52.3, 79.8)
- added R4: 100, Resistor_THT:R_Axial_DIN0204_L3.6mm_D1.6mm_P5.08mm_Horizontal, F.Cu at (101.6, 83.3)
- added R5: 100, Resistor_THT:R_Axial_DIN0204_L3.6mm_D1.6mm_P5.08mm_Horizontal, F.Cu at (101.6, 79.8)
- added R6: 100, Resistor_THT:R_Axial_DIN0204_L3.6mm_D1.6mm_P5.08mm_Horizontal, F.Cu at (149.9, 83.3)
- added R7: 100, Resistor_THT:R_Axial_DIN0204_L3.6mm_D1.6mm_P5.08mm_Horizontal, F.Cu at (149.9, 79.8)
- added R8: 100, Resistor_THT:R_Axial_DIN0204_L3.6mm_D1.6mm_P5.08mm_Horizontal, F.Cu at (198.6, 83.3)
- added R9: 100, Resistor_THT:R_Axial_DIN0204_L3.6mm_D1.6mm_P5.08mm_Horizontal, F.Cu at (198.6, 79.8)
- C1, C2, C3, C4, C5: value C -> 47uF
- J2: footprint Connector_USB:USB_B_Amphenol_MUSB-D511_Vertical_Rugged -> library:USB_2_0
- R1: value R -> 100
- SW1: footprint Button_Switch_THT:SW_E-Switch_EG1224_SPDT_Angled -> CKN10397-ND
- moved R1 11.2 mm to (47.3, 74.2), turned to 0 degrees
- moved C1 7.95 mm to (97.3, 52.2), turned to 270 degrees
- moved C2 7.94 mm to (145.7, 52.2), turned to 270 degrees
- moved C3 7.86 mm to (194.1, 52.2), turned to 270 degrees
- moved C4 7.62 mm to (243.0, 52.1), turned to 270 degrees
- moved C5 7.57 mm to (291.0, 52.3), turned to 270 degrees
- moved SW1 5.42 mm to (42.2, 72.2)
- moved J2 5.00 mm to (48.3, 56.9), turned to 270 degrees
- moved SW5 4.06 mm to (238.8, 42.7)
- moved SW6 4.06 mm to (287.0, 42.7)
- moved SW2 4.06 mm to (94.0, 42.7)
- moved SW3 4.06 mm to (142.2, 42.7)
- moved SW4 4.06 mm to (190.5, 42.7)
- moved J10 2.54 mm to (280.9, 51.3)
- moved J11 2.54 mm to (232.7, 51.3)
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Connections:
- J1 pad 13: Net-(J1-Pad13) -> LED1
- J1 pad 14: Net-(J1-Pad14) -> LED2
- J1 pad 7: Net-(J1-Pad7) -> GND
- J10 pad 8: Net-(J10-Pad8) -> GND
- J11 pad 8: Net-(J11-Pad8) -> GND
- J3 pad 8: Net-(J3-Pad8) -> GND
- J4 pad 13: Net-(J4-Pad13) -> LED3
- J4 pad 14: Net-(J4-Pad14) -> LED4
- J4 pad 7: Net-(J4-Pad7) -> GND
- J5 pad 8: Net-(J5-Pad8) -> GND
- J6 pad 13: Net-(J6-Pad13) -> LED5
- J6 pad 14: Net-(J6-Pad14) -> LED6
- J6 pad 7: Net-(J6-Pad7) -> GND
- J7 pad 8: Net-(J7-Pad8) -> GND
- J8 pad 13: Net-(J8-Pad13) -> LED9
- J8 pad 14: Net-(J8-Pad14) -> LED10
- J8 pad 7: Net-(J8-Pad7) -> GND
- J9 pad 13: Net-(J9-Pad13) -> LED7
- J9 pad 14: Net-(J9-Pad14) -> LED8
- J9 pad 7: Net-(J9-Pad7) -> GND
Routing:
- net Net-(J10-Pad3): track 32.3 -> 23.1 mm
- net Net-(J11-Pad3): track 31.7 -> 23.4 mm
- net LED1: track 0.00 -> 7.87 mm
- net Net-(J3-Pad3): track 30.4 -> 23.0 mm
- net LED2: track 0.00 -> 7.02 mm
- net LED5: track 0.00 -> 6.85 mm
- net LED3: track 0.00 -> 6.85 mm
- net LED7: track 0.00 -> 6.85 mm
- net LED6: track 0.00 -> 6.01 mm
- net LED4: track 0.00 -> 6.01 mm
- net LED8: track 0.00 -> 6.01 mm
- net LED9: track 0.00 -> 5.83 mm
- net Net-(J5-Pad3): track 30.1 -> 24.4 mm
- net LED10: track 0.00 -> 4.99 mm
- net Net-(D5-Pad1): track 0.00 -> 4.98 mm
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Other:
- board size 264.2 x 52.8 mm -> 267.7 x 52.9 mm
- rule trace_min: 0.2 -> 0.1778
- rule via_min_size: 0.4 -> 0.381

Commit message: fixed switches
Parts:
- SW2, SW3, SW4, SW5, SW6: footprint Button_Switch_THT:SW_PUSH_6mm -> library:SW_TH_Tactile_Omron_B3F-10xx
- moved SW2 25.4 mm to (94.0, 68.1)
- moved SW3 25.4 mm to (142.2, 68.1)
- moved SW4 25.4 mm to (190.5, 68.1)
- moved SW5 25.4 mm to (238.8, 68.1)
- moved SW6 25.4 mm to (287.0, 68.1)
- moved SW1 18.4 mm to (44.6, 54.0)
- moved R1 18.3 mm to (48.5, 56.0)
- moved J2 11.6 mm to (47.7, 68.5)
Routing:
- net Net-(J5-Pad3): track 24.4 -> 19.5 mm
- net Net-(J3-Pad3): track 23.0 -> 18.1 mm
- net Net-(J11-Pad3): track 23.4 -> 19.0 mm
- net Net-(J10-Pad3): track 23.1 -> 18.7 mm
- net Net-(J7-Pad3): track 23.3 -> 19.0 mm
- net Net-(J2-Pad1): track 24.7 -> 22.1 mm
- net Net-(R1-Pad1): track 5.16 -> 3.91 mm
Other:
- outline, holes or cut-outs redrawn

Commit message: updated foorprints
Parts:
- R1, R10, R11, R2, R3, R4, R5, R6, R7, R8, R9: footprint Resistor_THT:R_Axial_DIN0204_L3.6mm_D1.6mm_P5.08mm_Horizontal -> Resistor_THT:R_Axial_DIN0204_L3.6mm_D1.6mm_P7.62mm_Horizontal
- SW1: footprint CKN10397-ND -> library:CKN10397-ND
- moved R2 1.22 mm to (52.3, 82.1)
- moved J6 1.02 mm to (160.5, 51.3)
- moved J8 1.02 mm to (257.0, 51.3)
- moved J1 1.02 mm to (64.0, 51.3)
- moved J4 1.02 mm to (112.3, 51.3)
- moved J9 1.02 mm to (208.8, 51.3)
- moved R3 0.99 mm to (52.3, 78.8)
- moved D10 0.26 mm to (250.7, 78.7)
- moved D9 0.26 mm to (250.7, 85.3)
- moved R10 0.26 mm to (247.7, 83.3)
- moved R11 0.26 mm to (247.7, 79.7)
Routing:
- net Net-(D1-Pad1): track 4.40 -> 5.63 mm
- net LED9: track 5.83 -> 6.87 mm
- net LED6: track 6.01 -> 4.99 mm
- net LED5: track 6.85 -> 5.83 mm
- net LED4: track 6.01 -> 4.99 mm
- net LED3: track 6.85 -> 5.83 mm
- net LED2: track 7.02 -> 6.01 mm
- net LED1: track 7.87 -> 6.85 mm
- net LED8: track 6.01 -> 4.99 mm
- net LED7: track 6.85 -> 5.83 mm
- net LED10: track 4.99 -> 4.21 mm

Commit message: seperated board to top and bottom
Parts:
- added J12: Conn_01x06_Female, Connector_PinHeader_2.54mm:PinHeader_1x02_P2.54mm_Vertical, F.Cu at (64.0, 73.9)
- added J13: Conn_01x06_Female, Connector_PinHeader_2.54mm:PinHeader_1x02_P2.54mm_Vertical, F.Cu at (87.9, 73.9)
- added J14: Conn_01x06_Female, Connector_PinHeader_2.54mm:PinHeader_1x02_P2.54mm_Vertical, F.Cu at (112.3, 73.9)
- added J15: Conn_01x06_Female, Connector_PinHeader_2.54mm:PinHeader_1x02_P2.54mm_Vertical, F.Cu at (136.1, 73.9)
- added J16: Conn_01x06_Female, Connector_PinHeader_2.54mm:PinHeader_1x02_P2.54mm_Vertical, F.Cu at (160.5, 73.9)
- added J17: Conn_01x06_Female, Connector_PinHeader_2.54mm:PinHeader_1x02_P2.54mm_Vertical, F.Cu at (184.3, 73.9)
- added J18: Conn_01x06_Female, Connector_PinHeader_2.54mm:PinHeader_1x02_P2.54mm_Vertical, F.Cu at (208.8, 73.9)
- added J19: Conn_01x06_Female, Connector_PinHeader_2.54mm:PinHeader_1x02_P2.54mm_Vertical, F.Cu at (232.7, 73.9)
- added J20: Conn_01x06_Female, Connector_PinHeader_2.54mm:PinHeader_1x02_P2.54mm_Vertical, F.Cu at (257.0, 73.9)
- added J21: Conn_01x06_Female, Connector_PinHeader_2.54mm:PinHeader_1x02_P2.54mm_Vertical, F.Cu at (280.9, 73.9)
- added J22: Conn_01x01_Female, Connector_PinHeader_1.00mm:PinHeader_1x01_P1.00mm_Vertical, F.Cu at (45.4, 73.1)
- added J23: Conn_01x01_Female, Connector_PinHeader_1.00mm:PinHeader_1x01_P1.00mm_Vertical, F.Cu at (45.3, 65.1)
- C1, C2, C3, C4, C5: footprint Capacitor_THT:CP_Radial_D8.0mm_P5.00mm -> Capacitor_THT:C_Disc_D4.3mm_W1.9mm_P5.00mm
- J1, J10, J11, J3, J4, J5, J6, J7, J8, J9: value Conn_01x15_Female -> Conn_01x06_Female; footprint Connector_PinHeader_2.54mm:PinHeader_1x15_P2.54mm_Vertical -> Connector_PinHeader_2.54mm:PinHeader_1x06_P2.54mm_Vertical
- R1: footprint Resistor_THT:R_Axial_DIN0204_L3.6mm_D1.6mm_P7.62mm_Horizontal -> Resistor_THT:R_Axial_DIN0207_L6.3mm_D2.5mm_P7.62mm_Horizontal
- moved J11 48.3 mm to (280.9, 51.3)
- moved J8 48.3 mm to (208.8, 51.3)
- moved J10 23.9 mm to (257.0, 51.3)
- moved J9 23.9 mm to (232.7, 51.3)
- moved J2 13.1 mm to (41.7, 56.9)
- moved MH2 12.5 mm to (38.1, 74.9)
- moved MH4 12.0 mm to (297.2, 74.9)
- moved R11 10.2 mm to (242.9, 70.7), turned to 0 degrees
- moved R1 9.86 mm to (57.3, 60.5), turned to 90 degrees
- moved R7 9.57 mm to (146.9, 70.7), turned to 0 degrees
- moved R5 9.54 mm to (98.7, 70.7), turned to 0 degrees
- moved R9 9.54 mm to (195.8, 70.7), turned to 0 degrees
- moved SW2 8.89 mm to (94.0, 59.2)
- moved SW3 8.89 mm to (142.2, 59.2)
- moved SW4 8.89 mm to (190.5, 59.2)
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Connections:
- J1 pad 1: Net-(J1-Pad1) -> (no net)
- J1 pad 3: Net-(J1-Pad3) -> (no net)
- J1 pad 4: Net-(J1-Pad4) -> (no net)
- J1 pad 5: Net-(J1-Pad5) -> (no net)
- J1 pad 6: Net-(J1-Pad6) -> (no net)
- J10 pad 1: VCC -> (no net)
- J10 pad 3: Net-(J10-Pad3) -> (no net)
- J10 pad 4: Net-(J10-Pad4) -> (no net)
- J10 pad 5: Net-(J10-Pad5) -> (no net)
- J10 pad 6: GND -> (no net)
- J11 pad 4: Net-(J11-Pad4) -> (no net)
- J11 pad 5: Net-(J11-Pad5) -> (no net)
- J11 pad 6: GND -> (no net)
- J2 pad 2: Net-(J2-Pad2) -> (no net)
- J2 pad 3: Net-(J2-Pad3) -> (no net)
- J3 pad 4: Net-(J3-Pad4) -> (no net)
- J3 pad 5: Net-(J3-Pad5) -> (no net)
- J3 pad 6: GND -> (no net)
- J4 pad 1: Net-(J4-Pad1) -> (no net)
- J4 pad 3: Net-(J4-Pad3) -> (no net)
- J4 pad 4: Net-(J4-Pad4) -> (no net)
- J4 pad 5: Net-(J4-Pad5) -> (no net)
- J4 pad 6: Net-(J4-Pad6) -> (no net)
- J5 pad 4: Net-(J5-Pad4) -> (no net)
- J5 pad 5: Net-(J5-Pad5) -> (no net)
- J5 pad 6: GND -> (no net)
- J6 pad 1: Net-(J6-Pad1) -> (no net)
- J6 pad 3: Net-(J6-Pad3) -> (no net)
- J6 pad 4: Net-(J6-Pad4) -> (no net)
- J6 pad 5: Net-(J6-Pad5) -> (no net)
- J6 pad 6: Net-(J6-Pad6) -> (no net)
- J7 pad 4: Net-(J7-Pad4) -> (no net)
- J7 pad 5: Net-(J7-Pad5) -> (no net)
- J7 pad 6: GND -> (no net)
- J8 pad 1: Net-(J8-Pad1) -> (no net)
- J8 pad 3: Net-(J8-Pad3) -> (no net)
- J8 pad 4: Net-(J8-Pad4) -> (no net)
- J8 pad 5: Net-(J8-Pad5) -> (no net)
- J8 pad 6: Net-(J8-Pad6) -> (no net)
- J9 pad 1: Net-(J9-Pad1) -> VCC
- J9 pad 4: Net-(J9-Pad4) -> (no net)
- J9 pad 5: Net-(J9-Pad5) -> (no net)
- J9 pad 6: Net-(J9-Pad6) -> (no net)
- SW5 pad 2: Net-(J11-Pad3) -> Net-(J9-Pad3)
- SW6 pad 2: Net-(J10-Pad3) -> Net-(J11-Pad3)
Routing:
- net Net-(J10-Pad3): track 18.7 -> 0.00 mm
- net Net-(J9-Pad3): track 0.00 -> 17.5 mm
- net Net-(J2-Pad1): track 22.1 -> 7.13 mm
- net LED5: track 5.83 -> 14.8 mm
- net LED1: track 6.85 -> 15.3 mm
- net LED3: track 5.83 -> 14.2 mm
- net LED9: track 6.87 -> 15.1 mm
- net LED7: track 5.83 -> 14.0 mm
- net Net-(D10-Pad1): track 3.47 -> 9.07 mm
- net Net-(D8-Pad1): track 3.47 -> 8.94 mm
- net Net-(D2-Pad1): track 3.59 -> 8.05 mm
- net Net-(D6-Pad1): track 3.98 -> 8.03 mm
- net Net-(D4-Pad1): track 3.98 -> 8.02 mm
- net LED10: track 4.21 -> 7.98 mm
- net Net-(J5-Pad3): track 19.5 -> 15.7 mm
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- added copper zone on F.Cu, net GND
- added copper zone on B.Cu, net VCC
- removed copper zone on B.Cu, net GND
- removed copper zone on F.Cu, net VCC
Other:
- board size 267.7 x 52.9 mm -> 274.1 x 41.5 mm
